Commit message: [modify] changing wheel link mass

File: URDF/ranger/ranger_mini_gazebo.urdf (robot description, URDF)
Before this commit: robot ranger_mini_v2, 9 links, 8 joints
Links:
- link fl_wheel_link: mass 8 -> 0.5
- link fr_wheel_link: mass 8 -> 0.5
- link rl_wheel_link: mass 8 -> 0.5
- link rr_wheel_link: mass 8 -> 0.5
